File: hardware/kicad/MeshCrossway_RevA.kicad_pcb (KiCad board)
At the start: 2 copper layers, 144 x 76.5 mm, 33 parts, among them J1 Waveshare ESP32-S3-Touch-LCD-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, J2 HOST DEBUG, J5 BATTERY JST-PH 2.0, U1 LOCAL 5V SOURCE — TBD, U2 XIAO + Wio-SX1262, U3 XIAO + Wio-SX1262, U4 Uputronics MAX-M10S 3V

Commit message: PCB: improve ground-plane continuity and signal routing
Routing:
- net /GNSS_PPS: vias 1 -> 0
Changed lines of the file:
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@@
 		(start 90 85)
 		(end 92.175 85)
-		(width 1)
-		(layer "B.Cu")
+		(width 0.25)
+		(layer "F.Cu")
 		(net "/MT_RADIO_TX")
 	)
@@
 		(start 89.88 85.12)
 		(end 90 85)
-		(width 1)
-		(layer "B.Cu")
+		(width 0.25)
+		(layer "F.Cu")
 		(net "/MT_RADIO_TX")
 	)
@@
 		(start 89.76 85.12)
 		(end 89.88 85.12)
-		(width 1)
-		(layer "B.Cu")
+		(width 0.25)
+		(layer "F.Cu")
 		(net "/MT_RADIO_TX")
 	)
@@
 		(start 100.825 85)
 		(end 104.88 85)
-		(width 1)
-		(layer "B.Cu")
+		(width 0.25)
+		(layer "F.Cu")
 		(net "/MT_RADIO_RX")
 	)
@@
 		(start 104.88 85)
 		(end 105 85.12)
-		(width 1)
-		(layer "B.Cu")
+		(width 0.25)
+		(layer "F.Cu")
 		(net "/MT_RADIO_RX")
 	)
@@
 		(start 106.46 131.98)
 		(end 106.46 130.03)
-		(width 1)
+		(width 0.5)
 		(layer "B.Cu")
 		(net "/J8_3V3")
@@
 		(start 106.12 131.98)
 		(end 106.46 131.98)
-		(width 1)
+		(width 0.5)
 		(layer "B.Cu")
 		(net "/J8_3V3")
@@
 		(start 106.46 130.03)
 		(end 105.785 129.355)
-		(width 1)
+		(width 0.5)
 		(layer "B.Cu")
 		(net "/J8_3V3")
@@
 		(start 105.785 129.355)
 		(end 105.785 123.48)
-		(width 1)
+		(width 0.5)
 		(layer "B.Cu")
 		(net "/J8_3V3")
@@
 		(end 209.5 85)
 		(width 0.25)
-		(layer "B.Cu")
+		(layer "F.Cu")
 		(net "/MC_RADIO_TX")
 	)
@@
 		(end 217.675 85)
 		(width 0.25)
-		(layer "B.Cu")
+		(layer "F.Cu")
 		(net "/MC_RADIO_TX")
 	)
@@
 		(end 224.62 85)
 		(width 0.25)
-		(layer "B.Cu")
+		(layer "F.Cu")
 		(net "/MC_RADIO_RX")
 	)
@@
 		(end 224.74 85.12)
 		(width 0.25)
-		(layer "B.Cu")
+		(layer "F.Cu")
 		(net "/MC_RADIO_RX")
 	)
@@
 		(net "/GNSS_PPS")
 	)
-	(via
-		(at 100.5 128)
-		(size 0.6)
-		(drill 0.3)
-		(layers "F.Cu" "B.Cu")
-		(free yes)
-		(net "/GNSS_PPS")
-	)
 	(segment
 		(start 100.345 128.155)
 		(end 100.5 128)
 		(width 0.25)
-		(layer "B.Cu")
+		(layer "F.Cu")
 		(net "/GNSS_PPS")
 	)
@@
 		(end 100.345 128.155)
 		(width 0.25)
-		(layer "B.Cu")
+		(layer "F.Cu")
 		(net "/GNSS_PPS")
 	)
@@
 		(start 98.96 129.805)
 		(end 98.96 129.9)
-		(width 1)
+		(width 0.25)
 		(layer "B.Cu")
 		(net "/GNSS_PPS_RAW")
@@
 		(start 98.96 129.9)
 		(end 101.04 131.98)
-		(width 1)
+		(width 0.25)
 		(layer "B.Cu")
 		(net "/GNSS_PPS_RAW")

Commit message: Update MeshCrossway_RevA.kicad_pcb
Routing:
- net /J8_3V3: track 115.4 -> 40.2 mm
- net /GNSS_PPS: track 52.4 -> 0.00 mm
- net /MT_HOST_TX: track 66.2 -> 105.3 mm, vias 0 -> 1
- net /MT_HOST_RX: track 76.0 -> 104.7 mm, vias 0 -> 1
- net /RADIO_A_5V: track 78.2 -> 59.4 mm
- net /MC_HOST_TX: track 86.5 -> 100.1 mm
- net /MC_HOST_RX: track 81.0 -> 94.5 mm

Commit message: Update MeshCrossway_RevA.kicad_pcb
Routing:
- net Net-(D1-A): track 125.7 -> 204.2 mm
- net /MC_HOST_TX: track 100.1 -> 87.3 mm, vias 0 -> 1
- net /MC_HOST_RX: track 94.5 -> 86.4 mm, vias 0 -> 1
- net /J8_5V: track 95.8 -> 95.1 mm

Commit message: Update MeshCrossway_RevA.kicad_pcb
Routing:
- net /J8_3V3: track 40.2 -> 112.8 mm
- net /GNSS_PPS: track 0.00 -> 72.3 mm, vias 0 -> 1
- net /GNSS_SCL: track 91.6 -> 99.6 mm
- net /GNSS_SDA: track 102.0 -> 109.2 mm
Changed lines of the file:
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@@
+	)
+	(segment
+		(start 106.12 131.98)
+		(end 107.64 133.5)
+		(width 0.5)
+		(layer "B.Cu")
+		(net "/J8_3V3")
+	)
+	(segment
+		(start 171.82 133.5)
+		(end 176.05 129.27)
+		(width 0.5)
+		(layer "B.Cu")
+		(net "/J8_3V3")
+	)
+	(segment
+		(start 107.64 133.5)
+		(end 171.82 133.5)
+		(width 0.5)
+		(layer "B.Cu")
+		(net "/J8_3V3")
 	)
 	(segment
@@
 	)
 	(segment
+		(start 176.05 129.45)
+		(end 176 129.5)
+		(width 0.25)
+		(layer "B.Cu")
+		(net "/J8_3V3")
+	)
+	(segment
 		(start 176.38 126.4)
 		(end 176.05 126.73)
@@
 	)
 	(segment
+		(start 176.05 129.27)
+		(end 176.05 129.45)
+		(width 0.25)
+		(layer "B.Cu")
+		(net "/J8_3V3")
+	)
+	(segment
 		(start 205.86 126.4)
 		(end 176.38 126.4)
@@
 		(layer "F.Cu")
 		(net "/BAT")
+	)
+	(segment
+		(start 141.3 125)
+		(end 119 125)
+		(width 0.25)
+		(layer "F.Cu")
+		(net "/GNSS_PPS")
+	)
+	(segment
+		(start 143.03 126.73)
+		(end 141.3 125)
+		(width 0.25)
+		(layer "F.Cu")
+		(net "/GNSS_PPS")
+	)
+	(segment
+		(start 109.5 134.5)
+		(end 90.5 134.5)
+		(width 0.25)
+		(layer "F.Cu")
+		(net "/GNSS_PPS")
+	)
+	(segment
+		(start 89 131.41)
+		(end 92.41 128)
+		(width 0.25)
+		(layer "F.Cu")
+		(net "/GNSS_PPS")
+	)
+	(segment
+		(start 89 133)
+		(end 89 131.41)
+		(width 0.25)
+		(layer "F.Cu")
+		(net "/GNSS_PPS")
+	)
+	(segment
+		(start 92.41 128)
+		(end 97.5 128)
+		(width 0.25)
+		(layer "F.Cu")
+		(net "/GNSS_PPS")
+	)
+	(segment
+		(start 90.5 134.5)
+		(end 89 133)
+		(width 0.25)
+		(layer "F.Cu")
+		(net "/GNSS_PPS")
+	)
+	(segment
+		(start 119 125)
+		(end 109.5 134.5)
+		(width 0.25)
+		(layer "F.Cu")
+		(net "/GNSS_PPS")
+	)
+	(via
+		(at 97.5 128)
+		(size 0.6)
+		(drill 0.3)
+		(layers "F.Cu" "B.Cu")
+		(net "/GNSS_PPS")
+	)
+	(segment
+		(start 97.5 128)
+		(end 98.805 128)
+		(width 0.25)
+		(layer "B.Cu")
+		(net "/GNSS_PPS")
+	)
+	(segment
+		(start 98.805 128)
+		(end 98.96 128.155)
+		(width 0.25)
+		(layer "B.Cu")
+		(net "/GNSS_PPS")
 	)
 	(segment
@@
 	)
 	(segment
-		(start 95.02 133.58)
-		(end 164.12 133.58)
-		(width 0.25)
-		(layer "B.Cu")
+		(start 143.572412 123)
+		(end 146.795 126.222588)
+		(width 0.25)
+		(layer "F.Cu")
+		(net "/GNSS_SCL")
+	)
+	(segment
+		(start 147.512588 130.495)
+		(end 167.205 130.495)
+		(width 0.25)
+		(layer "F.Cu")
 		(net "/GNSS_SCL")
 	)
 	(segment
 		(start 93.42 131.98)
-		(end 95.02 133.58)
-		(width 0.25)
-		(layer "B.Cu")
+		(end 94.645 133.205)
+		(width 0.25)
+		(layer "F.Cu")
+		(net "/GNSS_SCL")
+	)
+	(segment
+		(start 146.795 129.777412)
+		(end 147.512588 130.495)
+		(width 0.25)
+		(layer "F.Cu")
+		(net "/GNSS_SCL")
+	)
+	(segment
+		(start 107.795 133.205)
+		(end 118 123)
+		(width 0.25)
+		(layer "F.Cu")
+		(net "/GNSS_SCL")
+	)
+	(segment
+		(start 167.205 130.495)
+		(end 168.43 129.27)
+		(width 0.25)
+		(layer "F.Cu")
+		(net "/GNSS_SCL")
+	)
+	(segment
+		(start 94.645 133.205)
+		(end 107.795 133.205)
+		(width 0.25)
+		(layer "F.Cu")
+		(net "/GNSS_SCL")
+	)
+	(segment
+		(start 146.795 126.222588)
+		(end 146.795 129.777412)
+		(width 0.25)
+		(layer "F.Cu")
+		(net "/GNSS_SCL")
+	)
+	(segment
+		(start 118 123)
+		(end 143.572412 123)
+		(width 0.25)
+		(layer "F.Cu")
 		(net "/GNSS_SCL")
 	)
@@
 	)
 	(segment
-		(start 164.12 133.58)
-		(end 168.43 129.27)
-		(width 0.25)
-		(layer "B.Cu")
-		(net "/GNSS_SCL")
-	)
-	(segment
 		(start 104.135 125.396667)
 		(end 98.730541 125.396667)
@@
 	)
 	(segment
-		(start 93.68 134.78)
-		(end 165.46 134.78)
-		(width 0.25)
-		(layer "B.Cu")
+		(start 142.032412 124)
+		(end 118.5 124)
+		(width 0.25)
+		(layer "F.Cu")
+		(net "/GNSS_SDA")
+	)
+	(segment
+		(start 108.5 134)
+		(end 92.9 134)
+		(width 0.25)
+		(layer "F.Cu")
+		(net "/GNSS_SDA")
+	)
+	(segment
+		(start 92.9 134)
+		(end 90.88 131.98)
+		(width 0.25)
+		(layer "F.Cu")
+		(net "/GNSS_SDA")
+	)
+	(segment
+		(start 144.345 126.312588)
+		(end 142.032412 124)
+		(width 0.25)
+		(layer "F.Cu")
+		(net "/GNSS_SDA")
+	)
+	(segment
+		(start 144.345 129.777412)
+		(end 144.345 126.312588)
+		(width 0.25)
+		(layer "F.Cu")
+		(net "/GNSS_SDA")
+	)
+	(segment
+		(start 118.5 124)
+		(end 108.5 134)
+		(width 0.25)
+		(layer "F.Cu")
+		(net "/GNSS_SDA")
+	)
+	(segment
+		(start 170.97 129.27)
+		(end 169.295 130.945)
+		(width 0.25)
+		(layer "F.Cu")
+		(net "/GNSS_SDA")
+	)
+	(segment
+		(start 169.295 130.945)
+		(end 145.512588 130.945)
+		(width 0.25)
+		(layer "F.Cu")
+		(net "/GNSS_SDA")
+	)
+	(segment
+		(start 145.512588 130.945)
+		(end 144.345 129.777412)
+		(width 0.25)
+		(layer "F.Cu")
 		(net "/GNSS_SDA")
 	)
@@
 	)
 	(segment
-		(start 165.46 134.78)
-		(end 170.97 129.27)
-		(width 0.25)
-		(layer "B.Cu")
-		(net "/GNSS_SDA")
-	)
-	(segment
 		(start 90.88 129.06)
 		(end 90.88 131.98)
@@
 		(width 0.25)
 		(layer "B.Cu")
-		(net "/GNSS_SDA")
-	)
-	(segment
-		(start 90.88 131.98)
-		(end 93.68 134.78)
-		(width 0.25)
-		(layer "B.Cu")
